File: ampli_ht.kicad_sch (KiCad schematic)
At the start: 29 parts, among them P201 CONN_2, P202 CONN_2, Q201 MPSA92, Q202 MPSA42, Q203 MPSA92, Q204 MPSA42, U201 LM358N

Commit message: Add ELDSGN parts + 'Popu test' variant for BOM mirror testing
Two parts from the ELDSGN parts DB placed in ampli_ht (hierarchical, 2
instances each): 00007 0603WAF6201T5E -> R1/R2, 00011 RC0402FR-07910RL2
-> R3/R4. Design variant 'Popu test' marks the R3 instance DNP.
Parts:
- added R1: 0603WAF6201T5E, connectors:C4260, symbol ELDSGN Parts:Resistors/00007 0603WAF6201T5E
- added R3: RC0402FR-07910RL2, connectors:C276279, symbol ELDSGN Parts:Resistors/00011 RC0402FR-07910RL2
Connections:
- net PIEZO_IN: now also R1.1
- net Vpil_0_3,3V: now also R3.2
- new net: R1.2, R3.1
