File: ampli_ht.kicad_sch (KiCad schematic)
At the start: 31 parts, among them P201 CONN_2, P202 CONN_2, Q201 MPSA92, Q202 MPSA42, Q203 MPSA92, Q204 MPSA42, U201 LM358N

Commit message: Repair ELDSGN parts for fixed dbl: flat lib_ids, no reserved-name fields (F-083/F-084)
De-slash 'ELDSGN Parts:Resistors/...' lib_ids (sub-library form KiCad
cannot resolve back), strip exclude_from_* fields (pcbnew skips any
component carrying that property key). Includes the stock-lib footprint
re-links from the earlier Update-PCB session.
Parts:
- added R5: 0603WAF6201T5E, connectors:C4260, symbol ELDSGN Parts:00007 0603WAF6201T5E
- R1: symbol ELDSGN Parts:Resistors/00007 0603WAF6201T5E -> ELDSGN Parts:00007 0603WAF6201T5E
- R3: symbol ELDSGN Parts:Resistors/00011 RC0402FR-07910RL2 -> ELDSGN Parts:00011 RC0402FR-07910RL2
Connections:
- net at R1.2, R3.1: now also R5.1
Other:
- moved on the sheet: R1
Changed lines of the file:
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@@
 	)
 	(junction
+		(at 74.93 96.52)
+		(diameter 0)
+		(color 0 0 0 0)
+	)
+	(junction
 		(at 185.42 83.82)
 		(diameter 1.016)
@@
 	(wire
 		(pts
+			(xy 93.98 118.11) (xy 74.93 118.11)
+		)
+		(stroke
+			(width 0)
+			(type default)
+		)
+	)
+	(wire
+		(pts
 			(xy 218.44 127) (xy 218.44 134.62)
 		)
@@
 	(wire
 		(pts
+			(xy 66.04 96.52) (xy 74.93 96.52)
+		)
+		(stroke
+			(width 0)
+			(type default)
+		)
+	)
+	(wire
+		(pts
 			(xy 72.39 50.8) (xy 78.74 50.8)
 		)
@@
 	(wire
 		(pts
-			(xy 55.88 96.52) (xy 53.34 96.52)
+			(xy 54.61 101.6) (xy 53.34 101.6)
 		)
 		(stroke
@@
 	(wire
 		(pts
-			(xy 53.34 50.8) (xy 53.34 96.52)
+			(xy 74.93 96.52) (xy 82.55 96.52)
+		)
+		(stroke
+			(width 0)
+			(type default)
+		)
+	)
+	(wire
+		(pts
+			(xy 53.34 50.8) (xy 53.34 101.6)
 		)
 		(stroke
@@
 	(wire
 		(pts
-			(xy 66.04 96.52) (xy 82.55 96.52)
+			(xy 64.77 101.6) (xy 66.04 101.6)
 		)
 		(stroke
@@
 	(wire
 		(pts
+			(xy 74.93 118.11) (xy 74.93 96.52)
+		)
+		(stroke
+			(width 0)
+			(type default)
+		)
+	)
+	(wire
+		(pts
 			(xy 226.06 137.16) (xy 226.06 162.56)
 		)
@@
 	(wire
 		(pts
+			(xy 66.04 101.6) (xy 66.04 96.52)
+		)
+		(stroke
+			(width 0)
+			(type default)
+		)
+	)
+	(wire
+		(pts
 			(xy 185.42 68.58) (xy 185.42 67.31)
 		)
@@
 	)
 	(symbol
-		(lib_id "ELDSGN Parts:Resistors/00007 0603WAF6201T5E")
-		(at 60.96 96.52 0)
+		(lib_id "ELDSGN Parts:00007 0603WAF6201T5E")
+		(at 99.06 118.11 0)
 		(unit 1)
 		(body_style 1)
@@
 		(dnp no)
 		(fields_autoplaced yes)
-		(property "Reference" "R1"
-			(at 60.96 90.17 0)
+		(property "Reference" "R5"
+			(at 99.06 111.76 0)
 			(show_name no)
 			(do_not_autoplace no)
@@
 		)
 		(property "Value" "0603WAF6201T5E"
-			(at 60.96 92.71 0)
+			(at 99.06 114.3 0)
 			(show_name no)
 			(do_not_autoplace no)
@@
 		)
 		(property "Footprint" "connectors:C4260"
-			(at 60.96 104.14 0)
+			(at 99.06 125.73 0)
 			(hide yes)
 			(show_name no)
@@
 		)
 		(property "Datasheet" "C21190.pdf"
-			(at 60.96 106.68 0)
+			(at 99.06 128.27 0)
 			(hide yes)
 			(show_name no)
@@
 		)
 		(property "Description" "Resistors"
-			(at 60.96 96.52 0)
+			(at 99.06 118.11 0)
 			(hide yes)
 			(show_name no)
@@
 		)
 		(property "LCSC Part" "C4260"
-			(at 60.96 109.22 0)
+			(at 99.06 130.81 0)
 			(hide yes)
 			(show_name no)
@@
 		)
 		(property "MPN" "0603WAF6201T5E"
-			(at 60.96 96.52 0)
+			(at 99.06 118.11 0)
 			(hide yes)
 			(show_name no)
@@
 		)
 		(property "Manufacturer" "UNI-ROYAL"
-			(at 60.96 96.52 0)
+			(at 99.06 118.11 0)
 			(hide yes)
 			(show_name no)
@@
 		)
 		(property "ELDSGN_id" "7"
-			(at 60.96 96.52 0)
+			(at 99.06 118.11 0)
 			(hide yes)
 			(show_name no)
@@
 		)
 		(property "ELDSGN_Category" ""
-			(at 60.96 96.52 0)
+			(at 99.06 118.11 0)
 			(hide yes)
 			(show_name no)
@@
 		)
 		(property "Package" ""
-			(at 60.96 96.52 0)
+			(at 99.06 118.11 0)
 			(hide yes)
 			(show_name no)
@@
 		)
 		(property "Power" ""
-			(at 60.96 96.52 0)
+			(at 99.06 118.11 0)
 			(hide yes)
 			(show_name no)
@@
 		)
 		(property "Resistance" ""
-			(at 60.96 96.52 0)
+			(at 99.06 118.11 0)
+			(hide yes)
+			(show_name no)
+			(do_not_autoplace no)
+			(effects
+				(font
+					(size 1.27 1.27)
+				)
+			)
+		)
+		(pin "2"
+		)
+		(pin "1"
+		)
+		(instances
+			(project "complex_hierarchy"
+				(path "/5b9623a5-6d01-41fc-9865-e1bc779418c8/00000000-0000-0000-0000-00004b3a1333"
+					(reference "R5")
+					(unit 1)
+				)
+				(path "/5b9623a5-6d01-41fc-9865-e1bc779418c8/00000000-0000-0000-0000-00004b3a13a4"
+					(reference "R6")
+					(unit 1)
+				)
+			)
+		)
+	)
+	(symbol
+		(lib_id "ELDSGN Parts:00007 0603WAF6201T5E")
+		(at 59.69 101.6 0)
+		(unit 1)
+		(body_style 1)
+		(exclude_from_sim no)
+		(in_bom yes)
+		(on_board yes)
+		(in_pos_files yes)
+		(dnp no)
+		(fields_autoplaced yes)
+		(property "Reference" "R1"
+			(at 59.69 95.25 0)
+			(show_name no)
+			(do_not_autoplace no)
+			(effects
+				(font
+					(size 1.27 1.27)
+				)
+			)
+		)
+		(property "Value" "0603WAF6201T5E"
+			(at 59.69 97.79 0)
+			(show_name no)
+			(do_not_autoplace no)
+			(effects
+				(font
+					(size 1.27 1.27)
+				)
+			)
+		)
+		(property "Footprint" "connectors:C4260"
+			(at 59.69 109.22 0)
 			(hide yes)
 			(show_name no)
@@
 			)
 		)
-		(property "exclude_from_board" ""
-			(at 60.96 96.52 0)
+		(property "Datasheet" "C21190.pdf"
+			(at 59.69 111.76 0)
 			(hide yes)
 			(show_name no)
@@
 			)
 		)
-		(property "exclude_from_bom" ""
-			(at 60.96 96.52 0)
+		(property "Description" "Resistors"
+			(at 59.69 101.6 0)
 			(hide yes)
 			(show_name no)
@@
 			)
 		)
-		(property "exclude_from_sim" ""
-			(at 60.96 96.52 0)
+		(property "LCSC Part" "C4260"
+			(at 59.69 114.3 0)
+			(hide yes)
+			(show_name no)
+			(do_not_autoplace no)
+			(effects
+				(font
+					(size 1.27 1.27)
+				)
+			)
+		)
+		(property "MPN" "0603WAF6201T5E"
+			(at 59.69 101.6 0)
+			(hide yes)
+			(show_name no)
+			(do_not_autoplace no)
+			(effects
+				(font
+					(size 1.27 1.27)
+				)
+			)
+		)
+		(property "Manufacturer" "UNI-ROYAL"
+			(at 59.69 101.6 0)
+			(hide yes)
+			(show_name no)
+			(do_not_autoplace no)
+			(effects
+				(font
+					(size 1.27 1.27)
+				)
+			)
+		)
+		(property "ELDSGN_id" "7"
+			(at 59.69 101.6 0)
+			(hide yes)
+			(show_name no)
+			(do_not_autoplace no)
+			(effects
+				(font
+					(size 1.27 1.27)
+				)
+			)
+		)
+		(property "ELDSGN_Category" ""
+			(at 59.69 101.6 0)
+			(hide yes)
+			(show_name no)
+			(do_not_autoplace no)
+			(effects
+				(font
+					(size 1.27 1.27)
+				)
+			)
+		)
+		(property "Package" ""
+			(at 59.69 101.6 0)
+			(hide yes)
+			(show_name no)
+			(do_not_autoplace no)
+			(effects
+				(font
+					(size 1.27 1.27)
+				)
+			)
+		)
+		(property "Power" ""
+			(at 59.69 101.6 0)
+			(hide yes)
+			(show_name no)
+			(do_not_autoplace no)
+			(effects
+				(font
+					(size 1.27 1.27)
+				)
+			)
+		)
+		(property "Resistance" ""
+			(at 59.69 101.6 0)
 			(hide yes)
 			(show_name no)
@@
 	)
 	(symbol
-		(lib_id "ELDSGN Parts:Resistors/00011 RC0402FR-07910RL2")
+		(lib_id "ELDSGN Parts:00011 RC0402FR-07910RL2")
 		(at 87.63 96.52 0)
 		(unit 1)
@@
 			(at 87.63 96.52 0)
 			(hide yes)
-			(show_name no)
-			(do_not_autoplace no)
-			(effects
-				(font
-					(size 1.27 1.27)
-				)
-			)
-		)
-		(property "exclude_from_board" ""
-			(at 87.63 96.52 0)
-			(hide yes)
-			(show_name no)
-			(do_not_autoplace no)
-			(effects
-				(font
-					(size 1.27 1.27)
-				)
-			)
-		)
-		(property "exclude_from_bom" ""
-			(at 87.63 96.52 0)
-			(hide yes)
-			(show_name no)
-			(do_not_autoplace no)
-			(effects
-				(font
-					(size 1.27 1.27)
-				)
-			)
-		)
-		(property "exclude_from_sim" ""
-			(at 87.63 96.52 0)
-			(hide yes)
