File: complex_hierarchy.kicad_pcb (KiCad board)
At the start: 2 copper layers, 100.7 x 80 mm, 68 parts, among them P101 CONN_2, P102 CONN_2, P201 CONN_2, P202 CONN_2, P301 CONN_2, P302 CONN_2, Q201 MPSA92, Q202 MPSA42, Q203 MPSA92, Q204 MPSA42, Q301 MPSA92, Q302 MPSA42, Q303 MPSA92, Q304 MPSA42, U101 78L05, U102 ICL7660, U201 LM358N, U301 LM358N

Commit message: Place R1-R6 on the board (assembly-test fixture for ELDSGN §16)
Parts:
- added R1: 0603WAF6201T5E, connectors:C4260, F.Cu at (201.5, 110.2)
- added R2: 0603WAF6201T5E, connectors:C4260, F.Cu at (201.5, 117.2)
- added R3: RC0402FR-07910RL2, connectors:C276279, F.Cu at (204.9, 110.1)
- added R4: RC0402FR-07910RL2, connectors:C276279, F.Cu at (204.9, 117.0)
- added R5: 0603WAF6201T5E, connectors:C4260, F.Cu at (201.5, 112.7)
- added R6: 0603WAF6201T5E, connectors:C4260, F.Cu at (201.5, 119.6)
- C101: footprint complex_hierarchy:CP_Axial_L11.0mm_D6.0mm_P18.00mm_Horizontal -> Capacitor_THT:CP_Axial_L11.0mm_D6.0mm_P18.00mm_Horizontal
- C102, C103, C104, C105: footprint complex_hierarchy:CP_Axial_L10.0mm_D4.5mm_P15.00mm_Horizontal -> Capacitor_THT:CP_Axial_L10.0mm_D4.5mm_P15.00mm_Horizontal
- C201, C202, C203, C204, C301, C302, C303, C304: footprint complex_hierarchy:C_Disc_D5.0mm_W2.5mm_P5.00mm -> Capacitor_THT:C_Disc_D5.0mm_W2.5mm_P5.00mm
- D101: footprint complex_hierarchy:D_DO-41_SOD81_P12.70mm_Horizontal -> Diode_THT:D_DO-41_SOD81_P12.70mm_Horizontal
- D201, D202, D203, D204, D301, D302, D303, D304: footprint complex_hierarchy:D_DO-35_SOD27_P7.62mm_Horizontal -> Diode_THT:D_DO-35_SOD27_P7.62mm_Horizontal
- P101, P102, P201, P202, P301, P302: footprint complex_hierarchy:Altech_AK300_1x02_P5.00mm_45-Degree -> TerminalBlock_Altech:Altech_AK300_1x02_P5.00mm_45-Degree
- Q201, Q202, Q203, Q204, Q301, Q302, Q303, U101: footprint complex_hierarchy:TO-92_HandSolder -> Package_TO_SOT_THT:TO-92_HandSolder
- R201, R202, R203, R204, R205, R206, R207, R208, R209, R210, R211, R212, R213, R301, R302, R303, R304, R305, R306, R307, R308, R309, R310, R311, R312, R313: footprint complex_hierarchy:R_Axial_DIN0204_L3.6mm_D1.6mm_P7.62mm_Horizontal -> Resistor_THT:R_Axial_DIN0204_L3.6mm_D1.6mm_P7.62mm_Horizontal
- RV201, RV301: footprint complex_hierarchy:Potentiometer_Bourns_3266W_Vertical -> Potentiometer_THT:Potentiometer_Bourns_3266W_Vertical
- U102, U201, U301: footprint complex_hierarchy:DIP-8_W7.62mm_LongPads -> Package_DIP:DIP-8_W7.62mm_LongPads
